Commit message: Add Create 2 description
Both Create 1 and Create 2 descriptions use the same base description. The mesh and some geometry (wheel size and axle length) vary between the two descriptions.
The Create 2 mesh originates from: https://github.com/goncabrita/roomba_robot

Since no Create platforms have gyros or lasers, the links and joints for these sensors have been removed.

File: create_description/urdf/create.urdf.xacro (robot description, xacro)
@@ -1,262 +1,7 @@
-<?xml version="1.0"?>
-<robot name="turtlebot_hardware" xmlns:xacro="http://ros.org/wiki/xacro">
-  <!-- Macro for TurtleBot body. Including Gazebo extensions, but does not include Kinect -->
-  <xacro:include filename="$(find create_description)/urdf/create_gazebo.urdf.xacro"/>
-  <xacro:property name="base_x" value="0.33" />
-  <xacro:property name="base_y" value="0.33" />
-	  <xacro:macro name="create">
-	    <material name="Green">
-	      <color rgba="0.0 0.8 0.0 1.0"/>
-	    </material>
-	  <!-- base_footprint is a fictitious link(frame) that is on the ground right below base_link origin, navigation stack depends on this frame -->
-	  <link name="base_footprint">
-	    <visual>
-	      <origin xyz="0 0 0" rpy="0 0 0" />
-	      <geometry>
-	        <box size="0.001 0.001 0.001" />
-	      </geometry>
-	      <material name="Green" />
-	    </visual>
-	    <collision>
-	      <origin xyz="0 0 0.017" rpy="0 0 0" />
-	      <geometry>
-	       <box size="0.001 0.001 0.001" />
-	      </geometry>
-	    </collision>
-	  </link>
-	  <link name="base_link">
-	    <inertial>
-	      <mass value="2" />
-	      <origin xyz="0 0 0.0" />
-	      <inertia ixx="0.01" ixy="0.0" ixz="0.0"
-	        iyy="0.01" iyz="0.0" izz="0.5" />
-	    </inertial>
-	    <visual>
-	      <origin xyz=" 0 0 0.0308" rpy="0 0 0" />
-	      <geometry>
-	        <mesh filename="package://create_description/meshes/create_body.dae"/>
-	      </geometry>
-	    </visual>
-	    <collision>
-	      <origin xyz="0.0 0.0 0.0308" rpy="0 0 0" />
-	      <geometry>
-	        <cylinder length="0.0611632" radius="0.16495"/>
-	      </geometry>
-	    </collision>
-	  </link>
-	  <link name="wall_sensor_link">
-	    <inertial>
-	      <mass value="0.01" />
-	      <origin xyz="0 0 0"/>
-	      <inertia ixx="0.001" ixy="0.0" ixz="0.0"
-	        iyy="0.001" iyz="0.0" izz="0.001" />
-	    </inertial>
-	  </link>
-	  <link name="left_cliff_sensor_link">
-	    <inertial>
-	      <mass value="0.01" />
-	      <origin xyz="0 0 0"/>
-	      <inertia ixx="0.001" ixy="0.0" ixz="0.0"
-	        iyy="0.001" iyz="0.0" izz="0.001" />
-	    </inertial>
-	  </link>
-	  <link name="right_cliff_sensor_link">
-	    <inertial>
-	      <mass value="0.01" />
-	      <origin xyz="0 0 0"/>
-	      <inertia ixx="0.001" ixy="0.0" ixz="0.0"
-	        iyy="0.001" iyz="0.0" izz="0.001" />
-	    </inertial>
-	  </link>
-	  <link name="leftfront_cliff_sensor_link">
-	    <inertial>
-	      <mass value="0.01" />
-	      <origin xyz="0 0 0"/>
-	      <inertia ixx="1.0" ixy="0.0" ixz="0.0"
-	        iyy="0.01" iyz="0.0" izz="0.01" />
-	    </inertial>
-	  </link>
-	  <link name="rightfront_cliff_sensor_link">
-	    <inertial>
-	      <mass value="0.01" />
-	      <origin xyz="0 0 0"/>
-	      <inertia ixx="0.001" ixy="0.0" ixz="0.0"
-	        iyy="0.001" iyz="0.0" izz="0.001" />
-	    </inertial>
-	  </link>
-	  <joint name="base_footprint_joint" type="fixed">
-	    <origin xyz="0 0 0.017" rpy="0 0 0" />
-	    <parent link="base_footprint"/>
-	    <child link="base_link" />
-	  </joint>
-	  <joint name="base_wall_sensor_joint" type="fixed">
-	    <origin xyz="0.09 -0.120 0.042" rpy="0 0 -1.0" />
-	    <parent link="base_link"/>
-	    <child link="wall_sensor_link" />
-	  </joint>
-	  <joint name="base_left_cliff_sensor_joint" type="fixed">
-	    <origin xyz="0.07 0.14 0.01" rpy="0 1.57079 0" />
-	    <parent link="base_link"/>
-	    <child link="left_cliff_sensor_link" />
-	  </joint>
-	  <joint name="base_right_cliff_sensor_joint" type="fixed">
-	    <origin xyz="0.07 -0.14 0.01" rpy="0 1.57079 0" />
-	    <parent link="base_link"/>
-	    <child link="right_cliff_sensor_link" />
-	  </joint>
-	  <joint name="base_leftfront_cliff_sensor_joint" type="fixed">
-	    <origin xyz="0.15 0.04 0.01" rpy="0 1.57079 0" />
-	    <parent link="base_link"/>
-	    <child link="leftfront_cliff_sensor_link" />
-	  </joint>
-	  <joint name="base_rightfront_cliff_sensor_joint" type="fixed">
-	    <origin xyz="0.15 -0.04 0.01" rpy="0 1.57079 0" />
-	    <parent link="base_link"/>
-	    <child link="rightfront_cliff_sensor_link" />
-	  </joint>
-	  <link name="left_wheel_link">
-	    <inertial>
-	      <origin xyz="0 0 0"/>
-	      <mass value="0.01" />
-	      <inertia ixx="0.001" ixy="0.0" ixz="0.0"
-	        iyy="0.001" iyz="0.0" izz="0.001" />
-	    </inertial>
-	    <visual>
-	      <origin xyz="0 0 0" rpy="0 1.5707 1.5707" />
-	      <geometry>
-	        <cylinder radius="0.033" length = "0.023"/>
-	      </geometry>
-	    </visual>
-	    <collision>
-	      <origin xyz="0 0 0" rpy="0 1.5707 1.5707" />
-	      <geometry>
-	        <cylinder radius="0.033" length = "0.023"/>
-	      </geometry>
-	    </collision>
-	  </link>
-	  <joint name="left_wheel_joint" type="continuous">
-	    <origin xyz="0 0.13 0.015" rpy="0 0 0"/>
-	    <parent link="base_link"/>
-	    <child link="left_wheel_link"/>
-	    <axis xyz="0 1 0"/>
-	  </joint>
-	  <link name="right_wheel_link">
-	    <inertial>
-	      <origin xyz="0 0 0"/>
-	      <mass value="0.01" />
-	      <inertia ixx="0.001" ixy="0.0" ixz="0.0"
-	        iyy="0.001" iyz="0.0" izz="0.001" />
-	    </inertial>
-	    <visual>
-	      <origin xyz="0 0 0" rpy="0 1.5707 1.5707" />
-	      <geometry>
-	        <cylinder radius="0.033" length = "0.023"/>
-	      </geometry>
-	    </visual>
-	    <collision>
-	      <origin xyz="0 0 0" rpy="0 1.5707 1.5707" />
-	      <geometry>
-	        <cylinder radius="0.033" length = "0.023"/>
-	      </geometry>
-	    </collision>
-	  </link>
-	  <joint name="right_wheel_joint" type="continuous">
-	    <origin xyz="0 -0.13 0.015" rpy="0 0 0"/>
-	    <parent link="base_link"/>
-	    <child link="right_wheel_link"/>
-	    <axis xyz="0 1 0"/>
-	  </joint>
-	  <link name="rear_wheel_link">
-	    <inertial>
-	      <origin xyz="0 0 0"/>
-	      <mass value="0.001" />
-	      <inertia ixx="0.0001" ixy="0.0" ixz="0.0"
-	        iyy="0.0001" iyz="0.0" izz="0.0001" />
-	    </inertial>
-	    <visual>
-	      <origin xyz="0 0 0" rpy="0 1.5707 1.5707"/>
-	      <geometry>
-	        <sphere radius="0.015" />
-	      </geometry>
-	    </visual>
-	    <collision>
-	      <origin xyz="0 0 0" rpy="0 1.5707 1.5707" />
-	      <geometry>
-	        <sphere radius="0.015" />
-	      </geometry>
-	    </collision>
-	  </link>
-	  <!-- fixed because there's no transmission -->
-	  <joint name="rear_castor_joint" type="fixed">
-	    <origin xyz="-0.13 0 0.0" rpy="0 0 0"/>
-	    <parent link="base_link"/>
-	    <child link="rear_wheel_link"/>
-	    <axis xyz="0 1 0"/>
-	  </joint>
-	  <link name="front_wheel_link">
-	    <inertial>
-	      <origin xyz="0 0 0" />
-	      <mass value="0.01" />
-	      <inertia ixx="0.001" ixy="0.0" ixz="0.0"
-	        iyy="0.001" iyz="0.0" izz="0.001" />
-	    </inertial>
-	    <visual>
-	      <origin xyz="0 0 0" rpy="0 1.5707 1.5707"/>
-	      <geometry>
-	        <sphere radius="0.018" />
-	      </geometry>
-	    </visual>
-	    <collision>
-	      <origin xyz="0 0 0" rpy="0 1.5707 1.5707" />
-	      <geometry>
-	        <sphere radius="0.018" />
-	      </geometry>
-	    </collision>
-	  </link>
-	  <!-- fixed because there's no transmission -->
-	  <joint name="front_castor_joint" type="fixed">
-	    <origin xyz="0.13 0 0.0" rpy="0 0 0"/>
-	    <parent link="base_link"/>
-	    <child link="front_wheel_link"/>
-	    <axis xyz="0 1 0"/>
-	  </joint>
-	  <joint name="gyro_joint" type="fixed">
-	    <axis xyz="0 1 0" />
-	    <origin xyz="0 0 0.04" rpy="0 0 0" />
-	    <parent link="base_link"/>
-	    <child link="gyro_link"/>
-	  </joint>
-	  <link name="gyro_link">
-	    <inertial>
-	      <mass value="0.001" />
-	      <origin xyz="0 0 0" rpy="0 0 0" />
-	      <inertia ixx="0.0001" ixy="0" ixz="0" iyy="0.000001" iyz="0" izz="0.0001" />
-	    </inertial>
-	  </link>
-	  <joint name="laser_joint" type="fixed">
-	    <origin xyz="-0.065 0 0.075" rpy="0 0 0" />
-	    <parent link="base_link" />
-	    <child link="laser" />
-	  </joint>
-	  <link name="laser">
-	    <visual>
-	      <geometry>
-	        <box size="0.02 0.035 0.002" />
-	      </geometry>
-	      <material name="Green" />
-	    </visual>
-	    <inertial>
-	      <mass value="0.001" />
-	      <origin xyz="0 0 0" />
-	      <inertia ixx="0.0001" ixy="0.0" ixz="0.0"
-	        iyy="0.0001" iyz="0.0"
-	        izz="0.0001" />
-	    </inertial>
-	  </link>
-	  <!-- Simulation sensors -->
-	  <sim_create/>
-	  <sim_create_wall_sensor/>
-	  <sim_create_cliff_sensors/>
-    <sim_imu/>
-  </xacro:macro>
+<?xml version="1.0" ?>
+<robot xmlns:xacro="http://ros.org/wiki/xacro" name="create">
+  <xacro:include filename="$(find create_description)/urdf/create_base.urdf.xacro" />
+  <xacro:create_base base_radius="0.3302" wheel_separation="0.26" wheel_radius="0.033">
+    <mesh filename="package://create_description/meshes/create_1.dae" />
+  </xacro:create_base>
 </robot>

File: create_description/urdf/create_base_gazebo.urdf.xacro (robot description, xacro)
@@ -1,20 +1,20 @@
-<?xml version="1.0"?>
-<robot xmlns:xacro="http://ros.org/wiki/xacro" name="turtlebot_gazebo">
-	<xacro:macro name="sim_create">
-	  <gazebo>
-	    <plugin name="create_controller" filename="libgazebo_ros_create.so">
-	      <alwaysOn>true</alwaysOn>
-	      <node_namespace>turtlebot_node</node_namespace>
-	      <left_wheel_joint>left_wheel_joint</left_wheel_joint>
-	      <right_wheel_joint>right_wheel_joint</right_wheel_joint>
-	      <front_castor_joint>front_castor_joint</front_castor_joint>
-	      <rear_castor_joint>rear_castor_joint</rear_castor_joint>
-	      <wheel_separation>.260</wheel_separation>
-	      <wheel_diameter>0.066</wheel_diameter>
-	      <base_geom>base_footprint_collision_base_link</base_geom>
-	      <updateRate>40</updateRate>
-	      <torque>1.0</torque>
-	    </plugin>
-	  </gazebo>
+<?xml version="1.0" ?>
+<robot xmlns:xacro="http://ros.org/wiki/xacro" name="create_base_gazebo">
+  <xacro:macro name="sim_create_base" params="wheel_diameter wheel_separation">
+    <gazebo>
+      <plugin name="create_controller" filename="libgazebo_ros_create.so">
+        <alwaysOn>true</alwaysOn>
+        <node_namespace>turtlebot_node</node_namespace>
+        <left_wheel_joint>left_wheel_joint</left_wheel_joint>
+        <right_wheel_joint>right_wheel_joint</right_wheel_joint>
+        <front_castor_joint>front_castor_joint</front_castor_joint>
+        <rear_castor_joint>rear_castor_joint</rear_castor_joint>
+        <wheel_separation>${wheel_separation}</wheel_separation>
+        <wheel_diameter>${wheel_diameter}</wheel_diameter>
+        <base_geom>base_footprint_collision_base_link</base_geom>
+        <updateRate>40</updateRate>
+        <torque>1.0</torque>
+      </plugin>
+    </gazebo>
     <gazebo reference="left_wheel_link">
       <mu1>1.0</mu1>
@@ -49,21 +49,7 @@
       <maxVel>1.0</maxVel>
     </gazebo>
-	</xacro:macro>
-	<xacro:macro name="sim_imu">
-	  <gazebo>
-	    <plugin name="imu_controller" filename="libgazebo_ros_imu.so">
-	      <alwaysOn>true</alwaysOn>
-	      <updateRate>30</updateRate>
-	      <bodyName>gyro_link</bodyName>
-	      <topicName>imu/data</topicName>
-        <serviceName>imu/is_calibrated</serviceName>
-	      <gaussianNoise>${0.0017*0.0017}</gaussianNoise>
-        <xyzOffsets>0 0 0</xyzOffsets>
-        <rpyOffsets>0 0 0</rpyOffsets>
-      </plugin>
-	  </gazebo>
-	</xacro:macro>
-	<xacro:macro name="sim_create_wall_sensor">
-	  <gazebo reference="wall_sensor_link">
+  </xacro:macro>
+  <xacro:macro name="sim_create_wall_sensor">
+    <gazebo reference="wall_sensor_link">
       <sensor type="ray" name="wall_sensor">
         <always_on>true</always_on>
@@ -87,8 +73,8 @@
         </ray>
       </sensor>
-	  </gazebo>
-	</xacro:macro>
-	<xacro:macro name="sim_create_cliff_sensors">
-	  <gazebo reference="left_cliff_sensor_link">
+    </gazebo>
+  </xacro:macro>
+  <xacro:macro name="sim_create_cliff_sensors">
+    <gazebo reference="left_cliff_sensor_link">
       <sensor type="ray" name="left_cliff_sensor">
         <always_on>true</always_on>
@@ -112,6 +98,6 @@
         </ray>
       </sensor>
-	  </gazebo>
-	  <gazebo reference="right_cliff_sensor_link">
+    </gazebo>
+    <gazebo reference="right_cliff_sensor_link">
       <sensor type="ray" name="right_cliff_sensor">
         <always_on>true</always_on>
@@ -135,6 +121,6 @@
         </ray>
       </sensor>
-	  </gazebo>
-	  <gazebo reference="leftfront_cliff_sensor_link">
+    </gazebo>
+    <gazebo reference="leftfront_cliff_sensor_link">
       <sensor type="ray" name="leftfront_cliff_sensor">
         <always_on>true</always_on>
@@ -158,6 +144,6 @@
         </ray>
       </sensor>
-	  </gazebo>
-	  <gazebo reference="rightfront_cliff_sensor_link">
+    </gazebo>
+    <gazebo reference="rightfront_cliff_sensor_link">
       <sensor type="ray" name="rightfront_cliff_sensor">
         <always_on>true</always_on>
@@ -181,5 +167,5 @@
         </ray>
       </sensor>
-	  </gazebo>
-	</xacro:macro>
+    </gazebo>
+  </xacro:macro>
 </robot>
